File: hardware/io.sch (EAGLE design)
At the start: 41 parts, among them IC1 LM2902D, IC2 LM2902D, U1 MMBT2222ALT1G, U2 MMBT2222ALT1G

Commit message: IO and Relay boards are distinct
Parts:
- removed D1: CGRM4001-G, diode:CGRM4001-G
- removed FAN: (no value), adafruit:PINHD-1X3
- removed HELED, PPLED: (no value), eagle-ltspice:LED_ESML0603
- removed R16, R9: 1K, resistor:R-US_R0402
- removed R17: 330, resistor:R-US_R1206
- removed R19, R20: 220, rcl:R-US_R0402
- removed U$1: T3050H-6I, digikey:T3050H-6I
- removed U$2: VM1-038-1AEHORIZONTAL, digikey:VM1-038-1AEHORIZONTAL
- removed U$3: G5LE-1A4_DC5, digikey:G5LE-1A4_DC5
- removed U$4: PC1725041, digikey:PC1725041
- removed U$5: MOC3020S, digikey:MOC3020S
- removed U$6: PC1719028, digikey:PC1719028
- removed U$7: CRM2512, digikey:CRM2512
- removed U1, U2: MMBT2222ALT1G, digikey:MMBT2222ALT1G
- added RELAYS: (no value), con-amp:MTA04-100
- HLT, MASH: device adafruit:PINHD-1X3 -> con-amp:MTA03-100
- PWR: value MTA-100-2HDR2 -> (none); device digikey:MTA-100-2HDR2 -> con-amp:MTA02-100
Connections:
- removed net +120: U$6.P$1, U$6.P$4
- removed net -120: U$1.A1, U$6.P$3
- removed net 120H: U$3.P$4, U$4.P$3
- removed net 120N: U$4.P$1, U$4.P$4
- removed net N$13: R17.1, U1.C
- removed net N$14: R17.2, U$5.CATHODE
- removed net N$15: R9.1, U1.B
- removed net N$16: R16.1, U2.B
- removed net N$18: D1.A, U$3.P$2, U2.C
- removed net N$19: U$1.G, U$5.OUT2
- removed net N$20: U$5.OUT1, U$7.P$1
- removed net N$22: U$1.A2, U$6.P$6, U$7.P$2
- removed net N$24: U$3.P$3, U$4.P$6
- removed net N$25: HELED.A, R19.2
- removed net N$26: PPLED.A, R20.2
- net +5V: now also PWR.2, RELAYS.1; no longer D1.C, FAN.2, PWR.A1, U$3.P$1, U$5.ANODE
- net GND: now also RELAYS.4; no longer FAN.1, HELED.C, PPLED.C, PWR.A2, U$4.P$2, U$4.P$5, U$6.P$5, U1.E, U2.E
- net HEOUT: now also RELAYS.2; no longer R19.1, R9.2
- net IN1: now also HLT.1; no longer HLT.3
- net IN2: now also MASH.1; no longer MASH.3
- net N$11: now also MASH.3; no longer MASH.1
- net N$12: now also HLT.3; no longer HLT.1
- net PPOUT: now also RELAYS.3; no longer R16.2, R20.1
